Commit message: trying to fix the gateway arm offset

File: gateway_description/xacro/big_arm_macro.xacro (robot description, xacro)
@@ -108,5 +108,6 @@
     <parent link="big_arm_link_0"/>
     <child link="big_arm_link_1"/>
-    <origin xyz="3.7698 0.3139 1.6058" rpy="0.0 -0.2094 -1.5708"/>
+    <!-- <origin xyz="3.7698 0.3139 1.6058" rpy="0.0 -0.2094 -1.5708"/> -->
+    <origin xyz="0.0 0.0 0.0" rpy="0.0 0.0 0.0"/>
   </joint>
   <joint name="big_arm_joint_2" type="revolute">

File: gateway_description/xacro/little_arm_macro.xacro (robot description, xacro)
@@ -120,5 +120,6 @@
     <parent link="little_arm_link_0"/>
     <child link="little_arm_link_1"/>
-    <origin xyz="13.984 -1.3352 -1.3367" rpy="2.3562 0.0 0.0"/>
+    <!-- <origin xyz="13.984 -1.3352 -1.3367" rpy="2.3562 0.0 0.0"/> -->
+    <origin xyz="0.0 0.0 0.0" rpy="0.0 0.0 0.0"/>
   </joint>
   <joint name="little_arm_joint_2" type="revolute">
