Commit message: urdf and xacros are making multi agent gateway via root links; static tf in launch for big and little arm to body

File: gateway_description/robots/big_arm.urdf.xacro (robot description, xacro)
@@ -2,6 +2,6 @@
 <robot xmlns:xacro="http://ros.org/wiki/xacro" name="big_arm">
   <xacro:include filename="$(find gateway_description)/xacro/big_arm_macro.xacro"/>
-  <link name="root"/>
-  <xacro:big_arm  parent="root">
+  <!-- <link name="gateway_body/root"/> -->
+  <xacro:big_arm>  <!-- parent="gateway_body/root"-->
     <origin xyz="0.0 0.0 0.0" rpy="0.0 0.4363 -1.396"/>
   </xacro:big_arm>

File: gateway_description/robots/little_arm.urdf.xacro (robot description, xacro)
@@ -2,6 +2,6 @@
 <robot xmlns:xacro="http://ros.org/wiki/xacro" name="little_arm">
   <xacro:include filename="$(find gateway_description)/xacro/little_arm_macro.xacro"/>
-  <link name="root"/>
-  <xacro:little_arm  parent="root">
+  <!-- <link name="gateway_body/root"/> -->
+  <xacro:little_arm> <!--  parent="gateway_body/root"-->
     <origin xyz="0.0 0.0 0.0" rpy="0.0 0.4363 -1.396"/>
   </xacro:little_arm>

File: gateway_description/xacro/big_arm_macro.xacro (robot description, xacro)
@@ -2,5 +2,5 @@
 <robot xmlns:xacro="http://ros.org/wiki/xacro" name="big_arm">
   <!-- BIG ARM -->
-  <xacro:macro name="big_arm" params=" parent:='' *origin ">
+  <xacro:macro name="big_arm" params=" *origin "> <!-- parent:=''-->
   <link name="big_arm_link_0"/>
   <link name="big_arm_link_1">
@@ -100,9 +100,9 @@
     </collision>
   </link>
-  <joint name="big_arm_joint_0" type="fixed">
+  <!-- <joint name="big_arm_joint_0" type="fixed">
     <parent link="${parent}"/>
     <child link="big_arm_link_0"/>
     <xacro:insert_block name="origin"/>
-  </joint>
+  </joint> -->
   <joint name="big_arm_joint_1" type="fixed">
     <parent link="big_arm_link_0"/>

File: gateway_description/xacro/little_arm_macro.xacro (robot description, xacro)
@@ -2,5 +2,5 @@
 <robot xmlns:xacro="http://ros.org/wiki/xacro" name="little_arm">
   <!-- LITTLE ARM -->
-  <xacro:macro name="little_arm" params=" parent:='' *origin ">
+  <xacro:macro name="little_arm" params=" *origin "> <!--parent:='' -->
   <link name="little_arm_link_0"/>
   <link name="little_arm_link_1">
@@ -112,9 +112,9 @@
     </collision>
   </link>
-  <joint name="little_arm_joint_0" type="fixed">
+  <!-- <joint name="little_arm_joint_0" type="fixed">
     <parent link="${parent}"/>
     <child link="little_arm_link_0"/>
     <xacro:insert_block name="origin"/>
-  </joint>
+  </joint> -->
   <joint name="little_arm_joint_1" type="fixed">
     <parent link="little_arm_link_0"/>

Commit message: fixed the gateway body sim to get the ros2 demo working

File: gateway_description/robots/big_arm.urdf.xacro (robot description, xacro)
@@ -2,6 +2,6 @@
 <robot xmlns:xacro="http://ros.org/wiki/xacro" name="big_arm">
   <xacro:include filename="$(find gateway_description)/xacro/big_arm_macro.xacro"/>
-  <!-- <link name="gateway_body/root"/> -->
-  <xacro:big_arm>  <!-- parent="gateway_body/root"-->
+  <link name="root"/>
+  <xacro:big_arm parent="root">
     <origin xyz="0.0 0.0 0.0" rpy="0.0 0.4363 -1.396"/>
   </xacro:big_arm>

File: gateway_description/robots/little_arm.urdf.xacro (robot description, xacro)
@@ -2,6 +2,6 @@
 <robot xmlns:xacro="http://ros.org/wiki/xacro" name="little_arm">
   <xacro:include filename="$(find gateway_description)/xacro/little_arm_macro.xacro"/>
-  <!-- <link name="gateway_body/root"/> -->
-  <xacro:little_arm> <!--  parent="gateway_body/root"-->
+  <link name="root"/>
+  <xacro:little_arm parent="root">
     <origin xyz="0.0 0.0 0.0" rpy="0.0 0.4363 -1.396"/>
   </xacro:little_arm>

File: gateway_description/xacro/big_arm_macro.xacro (robot description, xacro)
@@ -2,5 +2,5 @@
 <robot xmlns:xacro="http://ros.org/wiki/xacro" name="big_arm">
   <!-- BIG ARM -->
-  <xacro:macro name="big_arm" params=" *origin "> <!-- parent:=''-->
+  <xacro:macro name="big_arm" params=" parent:='' *origin ">
   <link name="big_arm_link_0"/>
   <link name="big_arm_link_1">
@@ -100,14 +100,13 @@
     </collision>
   </link>
-  <!-- <joint name="big_arm_joint_0" type="fixed">
+  <joint name="big_arm_joint_0" type="fixed">
     <parent link="${parent}"/>
     <child link="big_arm_link_0"/>
     <xacro:insert_block name="origin"/>
-  </joint> -->
+  </joint>
   <joint name="big_arm_joint_1" type="fixed">
     <parent link="big_arm_link_0"/>
     <child link="big_arm_link_1"/>
-    <!-- <origin xyz="3.7698 0.3139 1.6058" rpy="0.0 -0.2094 -1.5708"/> -->
-    <origin xyz="0.0 0.0 0.0" rpy="0.0 0.0 0.0"/>
+    <origin xyz="3.7698 0.3139 1.6058" rpy="0.0 -0.2094 -1.5708"/>
   </joint>
   <joint name="big_arm_joint_2" type="revolute">

File: gateway_description/xacro/little_arm_macro.xacro (robot description, xacro)
@@ -2,5 +2,5 @@
 <robot xmlns:xacro="http://ros.org/wiki/xacro" name="little_arm">
   <!-- LITTLE ARM -->
-  <xacro:macro name="little_arm" params=" *origin "> <!--parent:='' -->
+  <xacro:macro name="little_arm" params=" parent:='' *origin ">
   <link name="little_arm_link_0"/>
   <link name="little_arm_link_1">
@@ -112,18 +112,18 @@
     </collision>
   </link>
-  <!-- <joint name="little_arm_joint_0" type="fixed">
+  <joint name="little_arm_joint_0" type="fixed">
     <parent link="${parent}"/>
     <child link="little_arm_link_0"/>
     <xacro:insert_block name="origin"/>
-  </joint> -->
+  </joint>
   <joint name="little_arm_joint_1" type="fixed">
     <parent link="little_arm_link_0"/>
     <child link="little_arm_link_1"/>
-    <!-- <origin xyz="13.984 -1.3352 -1.3367" rpy="2.3562 0.0 0.0"/> -->
-    <origin xyz="0.0 0.0 0.0" rpy="0.0 0.0 0.0"/>
+    <origin xyz="13.984 -1.3352 -1.3367" rpy="2.3562 0.0 0.0"/>
   </joint>
   <joint name="little_arm_joint_2" type="revolute">
     <parent link="little_arm_link_1"/>
     <child link="little_arm_link_2"/>
+    <origin xyz="0.44043 0.010424 0.29487" rpy="0.0 0.0 0.0"/>
     <axis xyz="1 0 0"/>
     <limit lower="-3.14" upper="3.14" velocity="3.1416" effort="100"/> <!-- MADE UP NUMBERS JUST FOR TESTING -->
